Commit message: updated

File: urdf/fish.urdf (robot description, URDF)
Before this commit: robot fish_hpurv, 3 links, 2 joints
Links:
- removed link link_p1
- removed link link_p2
- added link imu_link, mass 0.1; collision box size=0.01 0.01 0.01; visual box size=0.01 0.01 0.01
- added link laser_frame, mass 0.1; collision cylinder length=0.04 radius=0.05; visual cylinder length=0.04 radius=0.05
- added link link_caudal, mass 0.2; collision mesh filename=$(find fish_hpurv)/meshes/link_caudal.stl; visual mesh filename=$(find fish_hpurv)/meshes/link_caudal.stl
- added link link_pectoral_left, mass 0.1; collision mesh filename=$(find fish_hpurv)/meshes/link_pectoral_left.stl; visual mesh filename=$(find fish_hpurv)/meshes/link_pectoral_left.stl
- added link link_pectoral_right, mass 0.1; collision mesh filename=$(find fish_hpurv)/meshes/link_pectoral_right.stl; visual mesh filename=$(find fish_hpurv)/meshes/link_pectoral_right.stl
- link link_base: mass 1e-09 -> 12; geometry collision mesh filename=$(find fish_hpurv)/meshes/link_base.stl; visual mesh filename=$(find fish_hpurv)/meshes/link_base.stl
Joints:
- added joint caudal_joint: type revolute, parent link_base, child link_caudal, origin xyz=0.425323 0.0953079 0.02 rpy=-1.5708 0 0, axis 0 0 1, limit lower=-0.523599 upper=0.523599 effort=10 velocity=10
- added joint imu_joint: type fixed, parent link_base, child imu_link, origin xyz=0.0325815 0.0493006 0.02 rpy=1.57 0 0
- added joint laser_joint: type fixed, parent link_base, child laser_frame, origin xyz=0.0325815 0.0493006 0.02 rpy=1.57 0 0
- joint joint1: child link_p2 -> link_pectoral_left; limit lower=-0.523599 upper=0.523599 effort=10 velocity=10 -> lower=-0.785398 upper=0.785398 effort=10 velocity=10; origin xyz=0.00565115 0.012105 0.0290034 rpy=3.14159 -0 0 -> xyz=-0.0504018 0.00224307 0.158572 rpy=3.14159 0 0
- joint joint2: child link_p1 -> link_pectoral_right; limit lower=-0.523599 upper=0.523599 effort=10 velocity=10 -> lower=-0.785398 upper=0.785398 effort=10 velocity=10; origin xyz=0.00565115 0.012105 -0.00238658 rpy=1.22465e-16 -0 0 -> xyz=-0.0504018 0.00224307 -0.120328 rpy=0 0 0

File: urdf/fish_hpurv_macro.urdf.xacro (robot description, xacro)
@@ -1,295 +1,384 @@
 <?xml version="1.0" ?>
 <robot name="fish_hpurv">
-  <!-- Link: link_base -->
-  <link name="link_base">
-    <inertial>
-      <origin xyz="0.0325815 0.0493006 -0.0204279" rpy="0 0 0"/>
-      <mass value="12"/>  <!-- assume base mass remains 12 kg -->
-      <inertia ixx="0.01" ixy="0" ixz="0" iyy="0.01" iyz="0" izz="0.01"/>
-    </inertial>
-    <visual>
-      <origin xyz="0.0325815 0.0493006 0.02" rpy="0 0 0"/>
-      <geometry>
-        <mesh filename="$(find fish_hpurv)/meshes/link_base.stl"/>
-      </geometry>
-      <material name="link_base_material">
-        <color rgba="0.796078 0.823529 0.937255 1.0"/>
-      </material>
-    </visual>
-    <collision>
-      <origin xyz="0.0325815 0.0493006 -0.0204279" rpy="0 0 0"/>
-      <geometry>
-        <mesh filename="$(find fish_hpurv)/meshes/link_base.stl"/>
-      </geometry>
-    </collision>
-  </link>
-  <!-- Link: link_caudal -->
-  <link name="link_caudal">
-    <inertial>
-      <origin xyz="-0.378805 2.04697e-16 -0.05" rpy="1.5708 0 0"/>
-      <mass value="0.2"/>
-      <inertia ixx="0.005" ixy="0" ixz="0" iyy="0.005" iyz="0" izz="0.005"/>
-    </inertial>
-    <visual>
-      <origin xyz="-0.378805 2.04697e-16 -0.05" rpy="1.5708 0 0"/>
-      <geometry>
-        <mesh filename="$(find fish_hpurv)/meshes/link_caudal.stl"/>
-      </geometry>
-      <material name="link_caudal_material">
-        <color rgba="0.796078 0.823529 0.937255 1.0"/>
-      </material>
-    </visual>
-    <collision>
-      <origin xyz="-0.378805 2.04697e-16 -0.05" rpy="1.5708 0 0"/>
-      <geometry>
-        <mesh filename="$(find fish_hpurv)/meshes/link_caudal.stl"/>
-      </geometry>
-    </collision>
-  </link>
-  <!-- Joint: caudal_joint (from link_base to link_caudal) -->
-  <joint name="caudal_joint" type="revolute">
-    <origin xyz="0.425323 0.0953079 0.02" rpy="-1.5708 0 0"/>
-    <parent link="link_base"/>
-    <child link="link_caudal"/>
-    <axis xyz="0 0 1"/>
-    <limit effort="10" velocity="10" lower="-0.523599" upper="0.523599"/>
-  </joint>
-  <!-- Link: link_pectoral_left -->
-  <link name="link_pectoral_left">
-    <inertial>
-      <origin xyz="0.0829833 -0.0470575 0.13" rpy="3.14159 0 0"/>
-      <mass value="0.1"/>
-      <inertia ixx="0.001" ixy="0" ixz="0" iyy="0.001" iyz="0" izz="0.001"/>
-    </inertial>
-    <visual>
-      <origin xyz="0.0829833 -0.0470575 0.13" rpy="3.14159 0 0"/>
-      <geometry>
-        <mesh filename="$(find fish_hpurv)/meshes/link_pectoral_left.stl"/>
-      </geometry>
-      <material name="link_pectoral_left_material">
-        <color rgba="0.796078 0.823529 0.937255 1.0"/>
-      </material>
-    </visual>
-    <collision>
-      <origin xyz="0.0829833 -0.0470575 0.13" rpy="3.14159 0 0"/>
-      <geometry>
-        <mesh filename="$(find fish_hpurv)/meshes/link_pectoral_left.stl"/>
-      </geometry>
-    </collision>
-  </link>
-  <!-- Joint: joint1 (from link_base to link_pectoral_left) -->
-  <joint name="joint1" type="revolute">
-    <origin xyz="-0.0504018 0.00224307 0.158572" rpy="3.14159 0 0"/>
-    <parent link="link_base"/>
-    <child link="link_pectoral_left"/>
-    <axis xyz="0 0 1"/>
-    <limit effort="10" velocity="10" lower="-0.785398" upper="0.785398"/>
-  </joint>
-  <!-- Link: link_pectoral_right -->
-  <link name="link_pectoral_right">
-    <inertial>
-      <origin xyz="0.0829833 0.0470575 0.13" rpy="0 0 0"/>
-      <mass value="0.1"/>
-      <inertia ixx="0.001" ixy="0" ixz="0" iyy="0.001" iyz="0" izz="0.001"/>
-    </inertial>
-    <visual>
-      <origin xyz="0.0829833 0.0470575 0.13" rpy="0 0 0"/>
-      <geometry>
-        <mesh filename="$(find fish_hpurv)/meshes/link_pectoral_right.stl"/>
-      </geometry>
-      <material name="link_pectoral_right_material">
-        <color rgba="0.796078 0.823529 0.937255 1.0"/>
-      </material>
-    </visual>
-    <collision>
-      <origin xyz="0.0829833 0.0470575 0.13" rpy="0 0 0"/>
-      <geometry>
-        <mesh filename="$(find fish_hpurv)/meshes/link_pectoral_right.stl"/>
-      </geometry>
-    </collision>
-  </link>
-  <!-- Joint: joint2 (from link_base to link_pectoral_right) -->
-  <joint name="joint2" type="revolute">
-    <origin xyz="-0.0504018 0.00224307 -0.120328" rpy="0 0 0"/>
-    <parent link="link_base"/>
-    <child link="link_pectoral_right"/>
-    <axis xyz="0 0 1"/>
-    <limit effort="10" velocity="10" lower="-0.785398" upper="0.785398"/>
-  </joint>
-  <joint name="laser_joint" type="fixed">
-    <parent link="link_base"/>
-    <child link="laser_frame"/>
-    <!-- Place the sensor slightly ahead; here we use an offset relative to link_base -->
-    <origin xyz="0.0325815 0.0493006 0.02" rpy="1.57 0 0"/>
-  </joint>
-  <link name="laser_frame">
-    <inertial>
-      <!-- The inertial origin is at (0,0,0) for the laser_frame -->
-      <origin xyz="0 0 0" rpy="0 0 0"/>
-      <mass value="0.1"/>
-      <inertia ixx="0.0001" ixy="0" ixz="0" iyy="0.0001" iyz="0" izz="0.0001"/>
-    </inertial>
-    <visual>
-      <origin xyz="0 0 0" rpy="0 0 0"/>
-      <geometry>
-        <cylinder radius="0.05" length="0.04"/>
-      </geometry>
-      <material name="red">
-        <color rgba="1 0 0 1"/>
-      </material>
-    </visual>
-    <collision>
-      <origin xyz="0 0 0" rpy="0 0 0"/>
-      <geometry>
-        <cylinder radius="0.05" length="0.04"/>
-      </geometry>
-    </collision>
-  </link>
-  <!-- Sensor plugin for the LiDAR remains as before -->
-  <gazebo reference="laser_frame">
-    <material>Gazebo/Red</material>
-    <sensor name="laser" type="ray">
-      <pose>0 0 0 0 0 0</pose>
-      <visualize>false</visualize>
-      <update_rate>10</update_rate>
-      <ray>
-        <scan>
-          <horizontal>
-            <samples>360</samples>
-            <min_angle>-3.14</min_angle>
-            <max_angle>3.14</max_angle>
-          </horizontal>
-        </scan>
-        <range>
-          <min>0.3</min>
-          <max>12</max>
-        </range>
-      </ray>
-      <plugin name="laser_controller" filename="libgazebo_ros_laser.so">
-        <ros>
-          <argument>~/out:=/scan</argument>
-        </ros>
-        <output_type>sensor_msgs/LaserScan</output_type>
-        <frame_name>laser_frame</frame_name>
-      </plugin>
-    </sensor>
-  </gazebo>
-  <joint name="imu_joint" type="fixed">
-    <parent link="link_base"/>
-    <child link="imu_link"/>
-    <!-- Place the IMU at a chosen offset on link_base; adjust xyz as needed -->
-    <origin xyz="0.0325815 0.0493006 0.02" rpy="1.57 0 0"/>
-  </joint>
-  <link name="imu_link">
-    <inertial>
-      <!-- Small inertial values for the sensor -->
-      <origin xyz="0 0 0" rpy="0 0 0"/>
-      <mass value="0.1"/>
-      <inertia ixx="0.000001" ixy="0" ixz="0" iyy="0.000001" iyz="0" izz="0.000001"/>
-    </inertial>
-    <visual>
-      <origin xyz="0 0 0" rpy="0 0 0"/>
-      <geometry>
-        <box size="0.01 0.01 0.01"/>
-      </geometry>
-      <material name="blue">
-        <color rgba="0 0 1 1"/>
-      </material>
-    </visual>
-    <collision>
-      <origin xyz="0 0 0" rpy="0 0 0"/>
-      <geometry>
-        <box size="0.01 0.01 0.01"/>
-      </geometry>
-    </collision>
-  </link>
-  <gazebo reference="imu_link">
-    <sensor name="imu_sensor" type="imu">
-      <update_rate>50</update_rate>
-      <always_on>true</always_on>
-      <visualize>true</visualize>
-      <plugin name="imu_plugin" filename="libgazebo_ros_imu.so">
-        <ros>
-          <argument>~/out:=/imu/data</argument>
-        </ros>
-        <topicName>/imu/data</topicName>
-        <frameName>imu_link</frameName>
-      </plugin>
-    </sensor>
-  </gazebo>
-<gazebo reference="link_base">
-  <sensor name="dvl_sensor" type="ray">
-    <!-- Sensor pose relative to link_base -->
-    <pose>0.03 -0.085 0  0  1.5708 0 </pose>
-    <!-- Enable visualization so you can see the beams -->
-    <visualize>true</visualize>
-    <!-- Set update rate (Hz) -->
-    <update_rate>10</update_rate>
-    <ray>
-      <scan>
-        <horizontal>
-          <!-- 360 samples for a full circle scan -->
-          <samples>360</samples>
-          <min_angle>3.14</min_angle>
-          <max_angle>6.28</max_angle>
-        </horizontal>
-      </scan>
-      <range>
-        <min>0.1</min>
-        <max>10</max>
-      </range>
-    </ray>
-    <!-- Load your custom DVL plugin -->
-    <plugin name="custom_dvl_plugin" filename="libfish_dvl_plugin.so"/>
-  </sensor>
-</gazebo>
-  <gazebo>
-    <!-- Buoyancy Plugin: Merge laser_frame into link_base -->
-    <plugin name="buoyancy_plugin" filename="libBuoyancyPlugin.so">
-      <fluid_density>1000</fluid_density>
-      <!-- For link_base, add the mass/volume of the laser_frame -->
-      <!-- Original link_base volume: 0.012; add 0.0001 from laser_frame = 0.0121 -->
-      <!-- The center of volume for link_base remains essentially unchanged -->
-      <link name="link_base">
-        <volume>0.0122</volume>
-        <center_of_volume>0.0325815 0.0493006 0.02</center_of_volume>
-      </link>
-      <link name="link_caudal">
-        <volume>0.0002</volume>
-        <center_of_volume>-0.378805 0  -0.05</center_of_volume>
-      </link>
-      <link name="link_pectoral_left">
-        <volume>0.0001</volume>
-        <center_of_volume>0.0829833 -0.0470575 0.13</center_of_volume>
-      </link>
-      <link name="link_pectoral_right">
-        <volume>0.0001</volume>
-        <center_of_volume>0.0829833 0.0470575 0.13</center_of_volume>
-      </link>
-      <!-- Remove the separate laser_frame entry so that its mass/volume is merged with link_base -->
-    </plugin>
-    <plugin name="hydrodynamics_plugin" filename="libHydrodynamicsPlugin.so">
-      <!-- Added mass terms (example values) -->
-      <xDotU>-10.0</xDotU>
-      <yDotV>-10.0</yDotV>
-      <zDotW>-10.0</zDotW>
-      <kDotP>-0.1</kDotP>
-      <mDotQ>-0.1</mDotQ>
-      <nDotR>-0.1</nDotR>
-      <!-- Linear and quadratic damping coefficients (example values) -->
-      <xUabsU>-0.32282</xUabsU>
-      <xU>-2.5</xU>
-      <yVabsV>-0.1</yVabsV>
-      <yV>-0.5</yV>
-      <zWabsW>-0.1</zWabsW>
-      <zW>-0.5</zW>
-      <kPabsP>-0.5</kPabsP>
-      <kP>-0.5</kP>
-      <mQabsQ>-0.5</mQabsQ>
-      <mQ>-0.5</mQ>
-      <nRabsR>-0.5</nRabsR>
-      <nR>-0.5</nR>
-      <default_current>0 0 0</default_current>
-    </plugin>
-  </gazebo>
+    <link name="link_base">
+    <inertial>
+      <origin xyz="0 0 0" rpy="0 0 0"/>
+      <mass value="0.1"/>
+      <inertia ixx="0.001" ixy="0" ixz="0" iyy="0.001" iyz="0" izz="0.001"/>
+    </inertial>
+        <visual>
+      <origin xyz="0 0 0" rpy="0 0 0"/>
+      <geometry>
+        <mesh filename="$(find fish_hpurv)/meshes/assets/part_8.stl"/>
+      </geometry>
+      <material name="part_8_material">
+        <color rgba="0.231373 0.380392 0.705882 1.0"/>
+      </material>
+    </visual>
+    <collision>
+      <origin xyz="0 0 0" rpy="0 0 0"/>
+      <geometry>
+        <mesh filename="$(find fish_hpurv)/meshes/assets/part_8.stl"/>
+      </geometry>
+    </collision>
+        <visual>
+      <origin xyz="0 0 0" rpy="0 0 0"/>
+      <geometry>
+        <mesh filename="$(find fish_hpurv)/meshes/assets/part_14.stl"/>
+      </geometry>
+      <material name="part_14_material">
+        <color rgba="0.615686 0.811765 0.929412 1.0"/>
+      </material>
+    </visual>
+    <collision>
+      <origin xyz="0 0 0" rpy="0 0 0"/>
+      <geometry>
+        <mesh filename="$(find fish_hpurv)/meshes/assets/part_14.stl"/>
+      </geometry>
+    </collision>
+        <visual>
+      <origin xyz="0 0 0" rpy="0 0 0"/>
+      <geometry>
+        <mesh filename="$(find fish_hpurv)/meshes/assets/part_20.stl"/>
+      </geometry>
+      <material name="part_20_material">
+        <color rgba="0.498039 0.498039 0.498039 1.0"/>
+      </material>
+    </visual>
+    <collision>
+      <origin xyz="0 0 0" rpy="0 0 0"/>
+      <geometry>
+        <mesh filename="$(find fish_hpurv)/meshes/assets/part_20.stl"/>
+      </geometry>
+    </collision>
+        <visual>
+      <origin xyz="0 0 0" rpy="0 0 0"/>
+      <geometry>
+        <mesh filename="$(find fish_hpurv)/meshes/assets/part_6.stl"/>
+      </geometry>
+      <material name="part_6_material">
+        <color rgba="0.615686 0.811765 0.929412 1.0"/>
+      </material>
+    </visual>
+    <collision>
+      <origin xyz="0 0 0" rpy="0 0 0"/>
+      <geometry>
+        <mesh filename="$(find fish_hpurv)/meshes/assets/part_6.stl"/>
+      </geometry>
+    </collision>
+        <visual>
+      <origin xyz="0 0 0" rpy="0 0 0"/>
+      <geometry>
+        <mesh filename="$(find fish_hpurv)/meshes/assets/part_18.stl"/>
+      </geometry>
+      <material name="part_18_material">
+        <color rgba="0.768627 0.886275 0.952941 1.0"/>
+      </material>
+    </visual>
+    <collision>
+      <origin xyz="0 0 0" rpy="0 0 0"/>
+      <geometry>
+        <mesh filename="$(find fish_hpurv)/meshes/assets/part_18.stl"/>
+      </geometry>
+    </collision>
+        <visual>
+      <origin xyz="0 0 0" rpy="0 0 0"/>
+      <geometry>
+        <mesh filename="$(find fish_hpurv)/meshes/assets/part_9.stl"/>
+      </geometry>
+      <material name="part_9_material">
+        <color rgba="0.917647 0.917647 0.917647 1.0"/>
+      </material>
+    </visual>
+    <collision>
+      <origin xyz="0 0 0" rpy="0 0 0"/>
+      <geometry>
+        <mesh filename="$(find fish_hpurv)/meshes/assets/part_9.stl"/>
+      </geometry>
+    </collision>
+        <visual>
+      <origin xyz="0 0 0" rpy="0 0 0"/>
+      <geometry>
+        <mesh filename="$(find fish_hpurv)/meshes/assets/part_16.stl"/>
+      </geometry>
+      <material name="part_16_material">
+        <color rgba="0.231373 0.380392 0.705882 1.0"/>
+      </material>
+    </visual>
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