Commit message: Initial commit

File: urdf/fish.urdf (robot description, URDF)
Before this commit: robot fish_hpurv, 6 links, 5 joints
Links:
- removed link imu_link
- removed link laser_frame
- removed link link_caudal
- removed link link_pectoral_left
- removed link link_pectoral_right
- added link link_hip, mass 10; collision mesh filename=$(find fish_hpurv)/mesh/assets/part_1.stl; collision mesh filename=$(find fish_hpurv)/mesh/assets/part_2.stl
- added link link_hip_2, mass 10; collision mesh filename=$(find fish_hpurv)/mesh/assets/part_1.stl; collision mesh filename=$(find fish_hpurv)/mesh/assets/part_2.stl
- added link link_hip_3, mass 10; collision mesh filename=$(find fish_hpurv)/mesh/assets/part_1.stl; collision mesh filename=$(find fish_hpurv)/mesh/assets/part_2.stl
- added link link_hip_4, mass 10; collision mesh filename=$(find fish_hpurv)/mesh/assets/part_1.stl; collision mesh filename=$(find fish_hpurv)/mesh/assets/part_2.stl
- added link link_thigh, mass 10; collision mesh filename=$(find fish_hpurv)/mesh/assets/part_2__2.stl; collision mesh filename=$(find fish_hpurv)/mesh/assets/part_3.stl
- added link link_thigh_2, mass 10; collision mesh filename=$(find fish_hpurv)/mesh/assets/part_2__2.stl; collision mesh filename=$(find fish_hpurv)/mesh/assets/part_3.stl
- added link link_thing_r, mass 10; collision mesh filename=$(find fish_hpurv)/mesh/assets/part_3__2.stl; collision mesh filename=$(find fish_hpurv)/mesh/assets/part_4__3.stl
- added link link_thing_r_2, mass 10; collision mesh filename=$(find fish_hpurv)/mesh/assets/part_3__2.stl; collision mesh filename=$(find fish_hpurv)/mesh/assets/part_4__3.stl
- link link_base: mass 12 -> 10; geometry collision mesh filename=$(find fish_hpurv)/mesh/assets/part_11.stl; collision mesh filename=$(find fish_hpurv)/mesh/assets/part_13.stl
Joints:
- removed joint caudal_joint
- removed joint imu_joint
- removed joint laser_joint
- added joint joint3: type revolute, parent link_hip, child link_hip_2, origin xyz=0 0 0 rpy=0 0 0, axis 0 0 1, limit lower=-3.141592653589793 upper=3.141592653589793 effort=10 velocity=10
- added joint joint4: type revolute, parent link_base, child link_hip_4, origin xyz=0 0 0 rpy=0 0 0, axis 0 0 1, limit lower=-3.141592653589793 upper=3.141592653589793 effort=10 velocity=10
- added joint joint5: type revolute, parent link_hip_4, child link_thigh_2, origin xyz=0 0 0 rpy=0 0 0, axis 0 0 1, limit lower=-3.141592653589793 upper=3.141592653589793 effort=10 velocity=10
- added joint joint6: type revolute, parent link_hip_2, child link_thigh, origin xyz=0 0 0 rpy=0 0 0, axis 0 0 1, limit lower=-3.141592653589793 upper=3.141592653589793 effort=10 velocity=10
- added joint joint7: type revolute, parent link_hip_3, child link_thing_r_2, origin xyz=0 0 0 rpy=0 0 0, axis 0 0 1, limit lower=-3.141592653589793 upper=3.141592653589793 effort=10 velocity=10
- added joint joint8: type revolute, parent link_hip, child link_thing_r, origin xyz=0 0 0 rpy=0 0 0, axis 0 0 1, limit lower=-3.141592653589793 upper=3.141592653589793 effort=10 velocity=10
- joint joint1: child link_pectoral_left -> link_hip; limit lower=-0.785398 upper=0.785398 effort=10 velocity=10 -> lower=-3.141592653589793 upper=3.141592653589793 effort=10 velocity=10; origin xyz=-0.0504018 0.00224307 0.158572 rpy=3.14159 0 0 -> xyz=0 0 0 rpy=0 0 0
- joint joint2: child link_pectoral_right -> link_hip_3; limit lower=-0.785398 upper=0.785398 effort=10 velocity=10 -> lower=-3.141592653589793 upper=3.141592653589793 effort=10 velocity=10; origin xyz=-0.0504018 0.00224307 -0.120328 rpy=0 0 0 -> xyz=0 0 0 rpy=0 0 0

File: urdf/fish_hpurv_macro.urdf.xacro (robot description, xacro)
@@ -1,9 +1,9 @@
 <?xml version="1.0" ?>
-<robot name="fish_hpurv">
+<robot name="robot">
     <link name="link_base">
     <inertial>
       <origin xyz="0 0 0" rpy="0 0 0"/>
-      <mass value="0.1"/>
-      <inertia ixx="0.001" ixy="0" ixz="0" iyy="0.001" iyz="0" izz="0.001"/>
+      <mass value="10"/>
+      <inertia ixx="1" ixy="0" ixz="0" iyy="1" iyz="0" izz="1"/>
     </inertial>
         <visual>
@@ -13,4 +13,64 @@
       </geometry>
       <material name="part_8_material">
+        <color rgba="0.768627 0.886275 0.952941 1.0"/>
+      </material>
+    </visual>
+    <collision>
+      <origin xyz="0 0 0" rpy="0 0 0"/>
+      <geometry>
+        <mesh filename="$(find fish_hpurv)/meshes/assets/part_8.stl"/>
+      </geometry>
+    </collision>
+        <visual>
+      <origin xyz="0 0 0" rpy="0 0 0"/>
+      <geometry>
+        <mesh filename="$(find fish_hpurv)/meshes/assets/part_4.stl"/>
+      </geometry>
+      <material name="part_4_material">
+        <color rgba="0.615686 0.811765 0.929412 1.0"/>
+      </material>
+    </visual>
+    <collision>
+      <origin xyz="0 0 0" rpy="0 0 0"/>
+      <geometry>
+        <mesh filename="$(find fish_hpurv)/meshes/assets/part_4.stl"/>
+      </geometry>
+    </collision>
+        <visual>
+      <origin xyz="0 0 0" rpy="0 0 0"/>
+      <geometry>
+        <mesh filename="$(find fish_hpurv)/meshes/assets/part_11.stl"/>
+      </geometry>
+      <material name="part_11_material">
+        <color rgba="0.980392 0.713725 0.00392157 1.0"/>
+      </material>
+    </visual>
+    <collision>
+      <origin xyz="0 0 0" rpy="0 0 0"/>
+      <geometry>
+        <mesh filename="$(find fish_hpurv)/meshes/assets/part_11.stl"/>
+      </geometry>
+    </collision>
+        <visual>
+      <origin xyz="0 0 0" rpy="0 0 0"/>
+      <geometry>
+        <mesh filename="$(find fish_hpurv)/meshes/assets/part_5.stl"/>
+      </geometry>
+      <material name="part_5_material">
+        <color rgba="0.647059 0.647059 0.647059 1.0"/>
+      </material>
+    </visual>
+    <collision>
+      <origin xyz="0 0 0" rpy="0 0 0"/>
+      <geometry>
+        <mesh filename="$(find fish_hpurv)/meshes/assets/part_5.stl"/>
+      </geometry>
+    </collision>
+        <visual>
+      <origin xyz="0 0 0" rpy="0 0 0"/>
+      <geometry>
+        <mesh filename="$(find fish_hpurv)/meshes/assets/part_14.stl"/>
+      </geometry>
+      <material name="part_14_material">
         <color rgba="0.231373 0.380392 0.705882 1.0"/>
       </material>
@@ -19,35 +79,20 @@
       <origin xyz="0 0 0" rpy="0 0 0"/>
       <geometry>
-        <mesh filename="$(find fish_hpurv)/meshes/assets/part_8.stl"/>
-      </geometry>
-    </collision>
-        <visual>
-      <origin xyz="0 0 0" rpy="0 0 0"/>
-      <geometry>
         <mesh filename="$(find fish_hpurv)/meshes/assets/part_14.stl"/>
       </geometry>
-      <material name="part_14_material">
-        <color rgba="0.615686 0.811765 0.929412 1.0"/>
-      </material>
-    </visual>
-    <collision>
-      <origin xyz="0 0 0" rpy="0 0 0"/>
-      <geometry>
-        <mesh filename="$(find fish_hpurv)/meshes/assets/part_14.stl"/>
-      </geometry>
-    </collision>
-        <visual>
-      <origin xyz="0 0 0" rpy="0 0 0"/>
-      <geometry>
-        <mesh filename="$(find fish_hpurv)/meshes/assets/part_20.stl"/>
-      </geometry>
-      <material name="part_20_material">
-        <color rgba="0.498039 0.498039 0.498039 1.0"/>
-      </material>
-    </visual>
-    <collision>
-      <origin xyz="0 0 0" rpy="0 0 0"/>
-      <geometry>
-        <mesh filename="$(find fish_hpurv)/meshes/assets/part_20.stl"/>
+    </collision>
+        <visual>
+      <origin xyz="0 0 0" rpy="0 0 0"/>
+      <geometry>
+        <mesh filename="$(find fish_hpurv)/meshes/assets/part_7.stl"/>
+      </geometry>
+      <material name="part_7_material">
+        <color rgba="0.917647 0.917647 0.917647 1.0"/>
+      </material>
+    </visual>
+    <collision>
+      <origin xyz="0 0 0" rpy="0 0 0"/>
+      <geometry>
+        <mesh filename="$(find fish_hpurv)/meshes/assets/part_7.stl"/>
       </geometry>
     </collision>
@@ -58,5 +103,5 @@
       </geometry>
       <material name="part_6_material">
-        <color rgba="0.615686 0.811765 0.929412 1.0"/>
+        <color rgba="0.231373 0.380392 0.705882 1.0"/>
       </material>
     </visual>
@@ -69,15 +114,15 @@
         <visual>
       <origin xyz="0 0 0" rpy="0 0 0"/>
-      <geometry>
-        <mesh filename="$(find fish_hpurv)/meshes/assets/part_18.stl"/>
-      </geometry>
-      <material name="part_18_material">
-        <color rgba="0.768627 0.886275 0.952941 1.0"/>
-      </material>
-    </visual>
-    <collision>
-      <origin xyz="0 0 0" rpy="0 0 0"/>
-      <geometry>
-        <mesh filename="$(find fish_hpurv)/meshes/assets/part_18.stl"/>
+      <geometry>t
+        <mesh filename="$(find fish_hpurv)/meshes/assets/part_15.stl"/>
+      </geometry>
+      <material name="part_15_material">
+        <color rgba="0.917647 0.917647 0.917647 1.0"/>
+      </material>
+    </visual>
+    <collision>
+      <origin xyz="0 0 0" rpy="0 0 0"/>
+      <geometry>
+        <mesh filename="$(find fish_hpurv)/meshes/assets/part_15.stl"/>
       </geometry>
     </collision>
@@ -88,5 +133,5 @@
       </geometry>
       <material name="part_9_material">
-        <color rgba="0.917647 0.917647 0.917647 1.0"/>
+        <color rgba="0.972549 0.529412 0.00392157 1.0"/>
       </material>
     </visual>
@@ -100,97 +145,7 @@
       <origin xyz="0 0 0" rpy="0 0 0"/>
       <geometry>
-        <mesh filename="$(find fish_hpurv)/meshes/assets/part_16.stl"/>
-      </geometry>
-      <material name="part_16_material">
-        <color rgba="0.231373 0.380392 0.705882 1.0"/>
-      </material>
-    </visual>
-    <collision>
-      <origin xyz="0 0 0" rpy="0 0 0"/>
-      <geometry>
-        <mesh filename="$(find fish_hpurv)/meshes/assets/part_16.stl"/>
-      </geometry>
-    </collision>
-        <visual>
-      <origin xyz="0 0 0" rpy="0 0 0"/>
-      <geometry>
-        <mesh filename="$(find fish_hpurv)/meshes/assets/part_5.stl"/>
-      </geometry>
-      <material name="part_5_material">
-        <color rgba="0.980392 0.713725 0.00392157 1.0"/>
-      </material>
-    </visual>
-    <collision>
-      <origin xyz="0 0 0" rpy="0 0 0"/>
-      <geometry>
-        <mesh filename="$(find fish_hpurv)/meshes/assets/part_5.stl"/>
-      </geometry>
-    </collision>
-        <visual>
-      <origin xyz="0 0 0" rpy="0 0 0"/>
-      <geometry>
-        <mesh filename="$(find fish_hpurv)/meshes/assets/part_2.stl"/>
-      </geometry>
-      <material name="part_2_material">
-        <color rgba="0.768627 0.886275 0.952941 1.0"/>
-      </material>
-    </visual>
-    <collision>
-      <origin xyz="0 0 0" rpy="0 0 0"/>
-      <geometry>
-        <mesh filename="$(find fish_hpurv)/meshes/assets/part_2.stl"/>
-      </geometry>
-    </collision>
-        <visual>
-      <origin xyz="0 0 0" rpy="0 0 0"/>
-      <geometry>
-        <mesh filename="$(find fish_hpurv)/meshes/assets/part_4.stl"/>
-      </geometry>
-      <material name="part_4_material">
-        <color rgba="0.498039 0.498039 0.498039 1.0"/>
-      </material>
-    </visual>
-    <collision>
-      <origin xyz="0 0 0" rpy="0 0 0"/>
-      <geometry>
-        <mesh filename="$(find fish_hpurv)/meshes/assets/part_4.stl"/>
-      </geometry>
-    </collision>
-        <visual>
-      <origin xyz="0 0 0" rpy="0 0 0"/>
-      <geometry>
-        <mesh filename="$(find fish_hpurv)/meshes/assets/part_11.stl"/>
-      </geometry>
-      <material name="part_11_material">
-        <color rgba="0.972549 0.529412 0.00392157 1.0"/>
-      </material>
-    </visual>
-    <collision>
-      <origin xyz="0 0 0" rpy="0 0 0"/>
-      <geometry>
-        <mesh filename="$(find fish_hpurv)/meshes/assets/part_11.stl"/>
-      </geometry>
-    </collision>
-        <visual>
-      <origin xyz="0 0 0" rpy="0 0 0"/>
-      <geometry>
-        <mesh filename="$(find fish_hpurv)/meshes/assets/part_10.stl"/>
-      </geometry>
-      <material name="part_10_material">
-        <color rgba="0.768627 0.886275 0.952941 1.0"/>
-      </material>
-    </visual>
-    <collision>
-      <origin xyz="0 0 0" rpy="0 0 0"/>
-      <geometry>
-        <mesh filename="$(find fish_hpurv)/meshes/assets/part_10.stl"/>
-      </geometry>
-    </collision>
-        <visual>
-      <origin xyz="0 0 0" rpy="0 0 0"/>
-      <geometry>
-        <mesh filename="$(find fish_hpurv)/meshes/assets/part_15.stl"/>
-      </geometry>
-      <material name="part_15_material">
+        <mesh filename="$(find fish_hpurv)/meshes/assets/part_13.stl"/>
+      </geometry>
+      <material name="part_13_material">
         <color rgba="0.647059 0.647059 0.647059 1.0"/>
       </material>
@@ -199,110 +154,5 @@
       <origin xyz="0 0 0" rpy="0 0 0"/>
       <geometry>
-        <mesh filename="$(find fish_hpurv)/meshes/assets/part_15.stl"/>
-      </geometry>
-    </collision>
-        <visual>
-      <origin xyz="0 0 0" rpy="0 0 0"/>
-      <geometry>
-        <mesh filename="$(find fish_hpurv)/meshes/assets/part_3.stl"/>
-      </geometry>
-      <material name="part_3_material">
-        <color rgba="0.972549 0.529412 0.00392157 1.0"/>
-      </material>
-    </visual>
-    <collision>
-      <origin xyz="0 0 0" rpy="0 0 0"/>
-      <geometry>
-        <mesh filename="$(find fish_hpurv)/meshes/assets/part_3.stl"/>
-      </geometry>
-    </collision>
-        <visual>
-      <origin xyz="0 0 0" rpy="0 0 0"/>
-      <geometry>
-        <mesh filename="$(find fish_hpurv)/meshes/assets/part_7.stl"/>
-      </geometry>
-      <material name="part_7_material">
-        <color rgba="0.647059 0.647059 0.647059 1.0"/>
-      </material>
-    </visual>
-    <collision>
-      <origin xyz="0 0 0" rpy="0 0 0"/>
-      <geometry>
-        <mesh filename="$(find fish_hpurv)/meshes/assets/part_7.stl"/>
-      </geometry>
-    </collision>
-        <visual>
-      <origin xyz="0 0 0" rpy="0 0 0"/>
-      <geometry>
-        <mesh filename="$(find fish_hpurv)/meshes/assets/part_17.stl"/>
-      </geometry>
-      <material name="part_17_material">
-        <color rgba="0.917647 0.917647 0.917647 1.0"/>
-      </material>
-    </visual>
-    <collision>
-      <origin xyz="0 0 0" rpy="0 0 0"/>
-      <geometry>
-        <mesh filename="$(find fish_hpurv)/meshes/assets/part_17.stl"/>
-      </geometry>
-    </collision>
-        <visual>
-      <origin xyz="0 0 0" rpy="0 0 0"/>
-      <geometry>
-        <mesh filename="$(find fish_hpurv)/meshes/assets/part_1.stl"/>
-      </geometry>
-      <material name="part_1_material">
-        <color rgba="0.917647 0.917647 0.917647 1.0"/>
-      </material>
-    </visual>
-    <collision>
-      <origin xyz="0 0 0" rpy="0 0 0"/>
-      <geometry>
-        <mesh filename="$(find fish_hpurv)/meshes/assets/part_1.stl"/>
-      </geometry>
-    </collision>
-        <visual>
-      <origin xyz="0 0 0" rpy="0 0 0"/>
-      <geometry>
         <mesh filename="$(find fish_hpurv)/meshes/assets/part_13.stl"/>
-      </geometry>
-      <material name="part_13_material">
-        <color rgba="0.980392 0.713725 0.00392157 1.0"/>
-      </material>
-    </visual>
-    <collision>
-      <origin xyz="0 0 0" rpy="0 0 0"/>
-      <geometry>
-        <mesh filename="$(find fish_hpurv)/meshes/assets/part_13.stl"/>
-      </geometry>
-    </collision>
-        <visual>
-      <origin xyz="0 0 0" rpy="0 0 0"/>
-      <geometry>
-        <mesh filename="$(find fish_hpurv)/meshes/assets/part_19.stl"/>
-      </geometry>
-      <material name="part_19_material">
-        <color rgba="0.972549 0.529412 0.00392157 1.0"/>
-      </material>
-    </visual>
-    <collision>
-      <origin xyz="0 0 0" rpy="0 0 0"/>
-      <geometry>
-        <mesh filename="$(find fish_hpurv)/meshes/assets/part_19.stl"/>
-      </geometry>
-    </collision>
-        <visual>
-      <origin xyz="0 0 0" rpy="0 0 0"/>
-      <geometry>
-        <mesh filename="$(find fish_hpurv)/meshes/assets/part_12.stl"/>
-      </geometry>
-      <material name="part_12_material">
-        <color rgba="0.498039 0.498039 0.498039 1.0"/>
-      </material>
-    </visual>
-    <collision>
-      <origin xyz="0 0 0" rpy="0 0 0"/>
-      <geometry>
-        <mesh filename="$(find fish_hpurv)/meshes/assets/part_12.stl"/>
       </geometry>
     </collision>
@@ -311,13 +161,13 @@
     <inertial>
       <origin xyz="0 0 0" rpy="0 0 0"/>
-      <mass value="0.1"/>
-      <inertia ixx="0.001" ixy="0" ixz="0" iyy="0.001" iyz="0" izz="0.001"/>
+      <mass value="10"/>
+      <inertia ixx="1" ixy="0" ixz="0" iyy="1" iyz="0" izz="1"/>
     </inertial>
         <visual>
       <origin xyz="0 0 0" rpy="0 0 0"/>
       <geometry>
-        <mesh filename="$(find fish_hpurv)/meshes/assets/part_2__2.stl"/>
-      </geometry>
-      <material name="part_2_2_material">
+        <mesh filename="$(find fish_hpurv)/meshes/assets/part_2.stl"/>
+      </geometry>
+      <material name="part_2_material">
         <color rgba="0.231373 0.380392 0.705882 1.0"/>
       </material>
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